Commit message: robot with lidar plugin in gazebo

File: robot_description/urdf/gazebo_world.xacro (robot description, xacro)
@@ -10,13 +10,16 @@
     <material>Gazebo/Grey</material>
 </gazebo>
-<gazebo reference="caster_wheel">
+  <gazebo reference="caster_wheel">
     <material>Gazebo/Grey</material>
-    <mu1 value="0.1"/>
-    <mu2 value="0.1"/>
-</gazebo>
+    <surface>
+      <friction>
+        <ode>
+          <mu>0.1</mu>
+          <mu2>0.1</mu2>
+        </ode>
+      </friction>
+    </surface>
+  </gazebo>
 <gazebo reference="camera_link">
-    <material>Gazebo/Red</material>
-</gazebo>
-<gazebo reference="lidar_link">
     <material>Gazebo/Red</material>
 </gazebo>
@@ -46,5 +49,4 @@
     </plugin>
     </gazebo>
-<!--
 <gazebo reference="lidar_link">
   <sensor name="lidar_sensor" type="ray">
@@ -81,4 +83,3 @@
   </sensor>
 </gazebo>
--->
 </robot>

Commit message: joystick code for real robot corrected and tested along with rpi code

File: robot_description/urdf/gazebo_world.xacro (robot description, xacro)
@@ -82,4 +82,36 @@
     </plugin>
   </sensor>
+<gazebo reference="camera_link">
+  <material>Gazebo/Red</material>
+  <sensor name="camera_sensor" type="camera">
+    <pose>0 0 0 0 0 0</pose>
+    <visualize>true</visualize>
+    <update_rate>30</update_rate>
+    <camera>
+      <horizontal_fov>1.3962634</horizontal_fov>
+      <image>
+        <width>640</width>
+        <height>480</height>
+        <format>R8G8B8</format>
+      </image>
+      <clip>
+        <near>0.1</near>
+        <far>100</far>
+      </clip>
+      <noise>
+        <type>gaussian</type>
+        <mean>0.0</mean>
+        <stddev>0.007</stddev>
+      </noise>
+    </camera>
+    <plugin name="camera_controller" filename="libgazebo_ros_camera.so">
+      <ros>
+        <remapping>image_raw:=/camera/image_raw</remapping>
+      </ros>
+      <camera_name>camera</camera_name>
+      <frame_name>camera_link</frame_name>
+    </plugin>
+  </sensor>
+</gazebo>
 </gazebo>
 </robot>
