Commit message: joy subscriber added with button for buzzer

File: robot_description/urdf/diff_robot.xacro (robot description, xacro)
@@ -6,5 +6,5 @@
   <link name="base_link">
     <inertial>
-      <mass value="1.0"/>
+      <mass value="10.0"/> <!--determines the weight therby the stability of bots-->
       <origin xyz="0 0 0.05"/>
       <inertia ixx="0.01" ixy="0.0" ixz="0.0" iyy="0.01" iyz="0.0" izz="0.01"/>
@@ -155,4 +155,6 @@
     <origin xyz="-0.1 0.175 0.01" rpy="0 0 1.57"/>
     <axis xyz="1 0 0"/>
+    <limit effort="10.0" velocity="20.0"/>
+    <dynamics damping="0.1" friction="0.1"/>
   </joint>
   <joint name="right_wheel_joint" type="continuous">
@@ -161,9 +163,11 @@
     <origin xyz="-0.1 -0.175 0.01" rpy="0 0 1.57"/>
     <axis xyz="1 0 0"/>
+    <limit effort="10.0" velocity="20.0"/>
+    <dynamics damping="0.1" friction="0.1"/>
   </joint>
   <joint name="caster_joint" type="fixed">
     <parent link="base_link"/>
     <child link="caster_wheel"/>
-    <origin xyz="0.0 0.0 -0.05" rpy="0 0 1.57"/>
+    <origin xyz="0.0 0.0 -0.04" rpy="0 0 1.57"/>
   </joint>
   <joint name="camera_joint" type="fixed">
